Commit message: muslos agregagos a main

File: bogobot_rviz/urdf/humanoid_links.xacro (robot description, xacro)
@@ -116,3 +116,19 @@
 		</link>
 	</xacro:macro>
+	<xacro:macro name="link_tigh" params="name x y z row pitch yaw">
+		<link name="${name}">
+			<collision>
+        		<origin xyz="${x} ${y} ${z}" rpy="${row} ${pitch} ${yaw}"  />
+        		<geometry>
+        			<box size="0.04 0.04 0.19"/>
+        		</geometry>
+    		</collision>
+			<visual>
+        		<origin xyz="${x} ${y} ${z}" rpy="${row} ${pitch} ${yaw}" />
+        		<geometry>
+        			<box size="0.04 0.04 0.19"/>
+        		</geometry>
+    		</visual>
+		</link>
+	</xacro:macro>
 </robot>

File: bogobot_rviz/urdf/humanoid_main.urdf (robot description, URDF)
Before this commit: robot Bogobot_V1, 11 links, 10 joints
Links:
- added link link_left_tight; collision box size=0.04 0.04 0.19; visual box size=0.04 0.04 0.19
- added link link_right_tight; collision box size=0.04 0.04 0.19; visual box size=0.04 0.04 0.19
Joints:
- added joint q11: type revolute, parent link_right_hip_motor, child link_right_tight, origin xyz=0 0 0 rpy=0 0 0, axis 0 1 0, limit lower=-6.283185307179586 upper=6.283185307179586 effort=2.5 velocity=5.76
- added joint q12: type revolute, parent link_left_hip_motor, child link_left_tight, origin xyz=0 0 0 rpy=0 0 0, axis 0 1 0, limit lower=-6.283185307179586 upper=6.283185307179586 effort=2.5 velocity=5.76

File: bogobot_rviz/urdf/humanoid_main.urdf.xacro (robot description, xacro)
@@ -16,7 +16,9 @@
     <xacro:hip_metal_link name="link_right_hip_metal" x = "0.0" y = "0.0" z = "-0.0175" row = "0" pitch = "0" yaw = "0"/>
     <xacro:motor_double_join name="link_right_hip_motor" x = "0.0" y = "0.0" z = "-0.0225" row = "0" pitch = "0" yaw = "0"/>
+    <xacro:link_tigh name="link_right_tight" x = "0.0" y = "0.0" z = "-0.085" row = "0" pitch = "0" yaw = "0"/>
     <!--pierna izquierda-->
     <xacro:hip_metal_link name="link_left_hip_metal" x = "0.0" y = "0.0" z = "-0.0175" row = "0" pitch = "0" yaw = "0"/>
     <xacro:motor_double_join name="link_left_hip_motor" x = "0.0" y = "0.0" z = "-0.0225" row = "0" pitch = "0" yaw = "0"/>
+    <xacro:link_tigh name="link_left_tight" x = "0.0" y = "0.0" z = "-0.085" row = "0" pitch = "0" yaw = "0"/>
     <!--JOINTS-->
     <!--hombro derecho-->
@@ -83,4 +85,11 @@
         <limit effort="2.5" lower="${-2*pi}" upper="${2*pi}" velocity="5.76"/>
     </joint>
+    <joint name="q11" type="revolute">
+        <origin rpy="0 0 0" xyz="0 0 0" />
+        <parent link="link_right_hip_motor" />
+        <child link="link_right_tight" />
+        <axis xyz="0 1 0" />
+        <limit effort="2.5" lower="${-2*pi}" upper="${2*pi}" velocity="5.76"/>
+    </joint>
     <!--pierna izquierda-->
     <joint name="q8" type="revolute">
@@ -98,3 +107,10 @@
         <limit effort="2.5" lower="${-2*pi}" upper="${2*pi}" velocity="5.76"/>
     </joint>
+    <joint name="q12" type="revolute">
+        <origin rpy="0 0 0" xyz="0 0 0" />
+        <parent link="link_left_hip_motor" />
+        <child link="link_left_tight" />
+        <axis xyz="0 1 0" />
+        <limit effort="2.5" lower="${-2*pi}" upper="${2*pi}" velocity="5.76"/>
+    </joint>
 </robot>

Commit message: ankle added

File: bogobot_rviz/urdf/humanoid_links.xacro (robot description, xacro)
@@ -132,3 +132,35 @@
 		</link>
 	</xacro:macro>
+	<xacro:macro name="link_knee" params="name x y z row pitch yaw">
+		<link name="${name}">
+			<collision>
+        		<origin xyz="${x} ${y} ${z}" rpy="${row} ${pitch} ${yaw}"  />
+        		<geometry>
+        			<box size="0.04 0.04 0.18"/>
+        		</geometry>
+    		</collision>
+			<visual>
+        		<origin xyz="${x} ${y} ${z}" rpy="${row} ${pitch} ${yaw}" />
+        		<geometry>
+        			<box size="0.04 0.04 0.18"/>
+        		</geometry>
+    		</visual>
+		</link>
+	</xacro:macro>
+	<xacro:macro name="foot" params="name x y z row pitch yaw">
+        <link name="${name}">
+            <collision>
+                <origin xyz="${x} ${y} ${z}" rpy="${row} ${pitch} ${yaw}" />
+                <geometry>
+                    <box size="0.15 0.2 0.01"/>
+                </geometry>
+            </collision>
+            <visual>
+                <origin xyz="${x} ${y} ${z}" rpy="${row} ${pitch} ${yaw}" />
+                <geometry>
+                    <box size="0.15 0.2 0.01"/>
+                </geometry>
+            </visual>
+        </link>
+    </xacro:macro>
 </robot>

File: bogobot_rviz/urdf/humanoid_main.urdf (robot description, URDF)
Before this commit: robot Bogobot_V1, 13 links, 12 joints
Links:
- removed link link_left_tight
- removed link link_right_tight
- added link link_left_knee; collision box size=0.04 0.04 0.18; visual box size=0.04 0.04 0.18
- added link link_left_tigh; collision box size=0.04 0.04 0.19; visual box size=0.04 0.04 0.19
- added link link_right_knee; collision box size=0.04 0.04 0.18; visual box size=0.04 0.04 0.18
- added link link_right_tigh; collision box size=0.04 0.04 0.19; visual box size=0.04 0.04 0.19
Joints:
- added joint q13: type revolute, parent link_right_tigh, child link_right_knee, origin xyz=0 0 -0.17 rpy=0 0 0, axis 0 1 0, limit lower=-6.283185307179586 upper=6.283185307179586 effort=2.5 velocity=5.76
- added joint q14: type revolute, parent link_left_tigh, child link_left_knee, origin xyz=0 0 -0.17 rpy=0 0 0, axis 0 1 0, limit lower=-6.283185307179586 upper=6.283185307179586 effort=2.5 velocity=5.76
- joint q11: child link_right_tight -> link_right_tigh
- joint q12: child link_left_tight -> link_left_tigh

File: bogobot_rviz/urdf/humanoid_main.urdf.xacro (robot description, xacro)
@@ -16,9 +16,12 @@
     <xacro:hip_metal_link name="link_right_hip_metal" x = "0.0" y = "0.0" z = "-0.0175" row = "0" pitch = "0" yaw = "0"/>
     <xacro:motor_double_join name="link_right_hip_motor" x = "0.0" y = "0.0" z = "-0.0225" row = "0" pitch = "0" yaw = "0"/>
-    <xacro:link_tigh name="link_right_tight" x = "0.0" y = "0.0" z = "-0.085" row = "0" pitch = "0" yaw = "0"/>
+    <xacro:link_tigh name="link_right_tigh" x = "0.0" y = "0.0" z = "-0.085" row = "0" pitch = "0" yaw = "0"/>
+    <xacro:link_knee name="link_right_knee" x = "0.0" y = "0.0" z = "-0.08" row = "0" pitch = "0" yaw = "0"/>
+    <!--xacro:motor_double_join name="link_right_ankle_motor" x = "0.0" y = "0.0" z = "0.0" row = "0" pitch = "0" yaw = "0"/-->
     <!--pierna izquierda-->
     <xacro:hip_metal_link name="link_left_hip_metal" x = "0.0" y = "0.0" z = "-0.0175" row = "0" pitch = "0" yaw = "0"/>
     <xacro:motor_double_join name="link_left_hip_motor" x = "0.0" y = "0.0" z = "-0.0225" row = "0" pitch = "0" yaw = "0"/>
-    <xacro:link_tigh name="link_left_tight" x = "0.0" y = "0.0" z = "-0.085" row = "0" pitch = "0" yaw = "0"/>
+    <xacro:link_tigh name="link_left_tigh" x = "0.0" y = "0.0" z = "-0.085" row = "0" pitch = "0" yaw = "0"/>
+    <xacro:link_knee name="link_left_knee" x = "0.0" y = "0.0" z = "-0.08" row = "0" pitch = "0" yaw = "0"/>
     <!--JOINTS-->
     <!--hombro derecho-->
@@ -88,8 +91,24 @@
         <origin rpy="0 0 0" xyz="0 0 0" />
         <parent link="link_right_hip_motor" />
-        <child link="link_right_tight" />
+        <child link="link_right_tigh" />
         <axis xyz="0 1 0" />
         <limit effort="2.5" lower="${-2*pi}" upper="${2*pi}" velocity="5.76"/>
     </joint>
+    <joint name="q13" type="revolute">
+        <origin rpy="0 0 0" xyz="0 0 -0.17" />
+        <parent link="link_right_tigh" />
+        <child link="link_right_knee" />
+        <axis xyz="0 1 0" />
+        <limit effort="2.5" lower="${-2*pi}" upper="${2*pi}" velocity="5.76"/>
+    </joint>
+    <!--
+    <joint name="q14" type="revolute">
+        <origin rpy="0 0 0" xyz="0 0 0" />
+        <parent link="link_right_tight" />
+        <child link="link_right_ankle_motor" />
+        <axis xyz="0 1 0" />
+        <limit effort="2.5" lower="${-2*pi}" upper="${2*pi}" velocity="5.76"/>
+    </joint>
+    -->
     <!--pierna izquierda-->
     <joint name="q8" type="revolute">
@@ -110,5 +129,12 @@
         <origin rpy="0 0 0" xyz="0 0 0" />
         <parent link="link_left_hip_motor" />
-        <child link="link_left_tight" />
+        <child link="link_left_tigh" />
+        <axis xyz="0 1 0" />
+        <limit effort="2.5" lower="${-2*pi}" upper="${2*pi}" velocity="5.76"/>
+    </joint>
+    <joint name="q14" type="revolute">
+        <origin rpy="0 0 0" xyz="0 0 -0.17" />
+        <parent link="link_left_tigh" />
+        <child link="link_left_knee" />
         <axis xyz="0 1 0" />
         <limit effort="2.5" lower="${-2*pi}" upper="${2*pi}" velocity="5.76"/>

Commit message: motor foot added

File: bogobot_rviz/urdf/humanoid_links.xacro (robot description, xacro)
@@ -148,4 +148,20 @@
 		</link>
 	</xacro:macro>
+	<xacro:macro name="motor_big_double_join" params="name x y z row pitch yaw">
+		<link name="${name}">
+			<collision>
+        		<origin xyz="${x} ${y} ${z}" rpy="${row} ${pitch} ${yaw}"  />
+        		<geometry>
+            			<box size="0.095 0.05 0.055"/>
+        		</geometry>
+    		</collision>
+			<visual>
+        		<origin xyz="${x} ${y} ${z}" rpy="${row} ${pitch} ${yaw}" />
+        		<geometry>
+            			<box size="0.095 0.05 0.055"/>
+        		</geometry>
+    		</visual>
+		</link>
+	</xacro:macro>
 	<xacro:macro name="foot" params="name x y z row pitch yaw">
         <link name="${name}">

File: bogobot_rviz/urdf/humanoid_main.urdf (robot description, URDF)
Before this commit: robot Bogobot_V1, 15 links, 14 joints
Links:
- added link link_left_ankle_motor; collision box size=0.095 0.05 0.055; visual box size=0.095 0.05 0.055
- added link link_right_ankle_motor; collision box size=0.095 0.05 0.055; visual box size=0.095 0.05 0.055
Joints:
- added joint q15: type revolute, parent link_right_knee, child link_right_ankle_motor, origin xyz=0 0 -0.16 rpy=0 0 0, axis 0 1 0, limit lower=-6.283185307179586 upper=6.283185307179586 effort=2.5 velocity=5.76
- added joint q16: type revolute, parent link_left_knee, child link_left_ankle_motor, origin xyz=0 0 -0.16 rpy=0 0 0, axis 0 1 0, limit lower=-6.283185307179586 upper=6.283185307179586 effort=2.5 velocity=5.76

File: bogobot_rviz/urdf/humanoid_main.urdf.xacro (robot description, xacro)
@@ -18,5 +18,5 @@
     <xacro:link_tigh name="link_right_tigh" x = "0.0" y = "0.0" z = "-0.085" row = "0" pitch = "0" yaw = "0"/>
     <xacro:link_knee name="link_right_knee" x = "0.0" y = "0.0" z = "-0.08" row = "0" pitch = "0" yaw = "0"/>
-    <!--xacro:motor_double_join name="link_right_ankle_motor" x = "0.0" y = "0.0" z = "0.0" row = "0" pitch = "0" yaw = "0"/-->
+    <xacro:motor_big_double_join name="link_right_ankle_motor" x = "-0.02625" y = "0.0" z = "0.02" row = "0" pitch = "0" yaw = "0"/>
     <!--pierna izquierda-->
     <xacro:hip_metal_link name="link_left_hip_metal" x = "0.0" y = "0.0" z = "-0.0175" row = "0" pitch = "0" yaw = "0"/>
@@ -24,4 +24,5 @@
     <xacro:link_tigh name="link_left_tigh" x = "0.0" y = "0.0" z = "-0.085" row = "0" pitch = "0" yaw = "0"/>
     <xacro:link_knee name="link_left_knee" x = "0.0" y = "0.0" z = "-0.08" row = "0" pitch = "0" yaw = "0"/>
+    <xacro:motor_big_double_join name="link_left_ankle_motor" x = "-0.02625" y = "0.0" z = "0.02" row = "0" pitch = "0" yaw = "0"/>
     <!--JOINTS-->
     <!--hombro derecho-->
@@ -102,13 +103,11 @@
         <limit effort="2.5" lower="${-2*pi}" upper="${2*pi}" velocity="5.76"/>
     </joint>
-    <!--
-    <joint name="q14" type="revolute">
-        <origin rpy="0 0 0" xyz="0 0 0" />
-        <parent link="link_right_tight" />
+    <joint name="q15" type="revolute">
+        <origin rpy="0 0 0" xyz="0 0 -0.16" />
+        <parent link="link_right_knee" />
         <child link="link_right_ankle_motor" />
         <axis xyz="0 1 0" />
         <limit effort="2.5" lower="${-2*pi}" upper="${2*pi}" velocity="5.76"/>
     </joint>
-    -->
     <!--pierna izquierda-->
     <joint name="q8" type="revolute">
@@ -140,3 +139,10 @@
         <limit effort="2.5" lower="${-2*pi}" upper="${2*pi}" velocity="5.76"/>
     </joint>
+    <joint name="q16" type="revolute">
+        <origin rpy="0 0 0" xyz="0 0 -0.16" />
+        <parent link="link_left_knee" />
+        <child link="link_left_ankle_motor" />
+        <axis xyz="0 1 0" />
+        <limit effort="2.5" lower="${-2*pi}" upper="${2*pi}" velocity="5.76"/>
+    </joint>
 </robot>

Commit message: foot link added

File: bogobot_rviz/urdf/humanoid_links.xacro (robot description, xacro)
@@ -169,5 +169,5 @@
                 <origin xyz="${x} ${y} ${z}" rpy="${row} ${pitch} ${yaw}" />
                 <geometry>
-                    <box size="0.15 0.2 0.01"/>
+                    <box size="0.2 0.15 0.01"/>
                 </geometry>
             </collision>
@@ -175,5 +175,5 @@
                 <origin xyz="${x} ${y} ${z}" rpy="${row} ${pitch} ${yaw}" />
                 <geometry>
-                    <box size="0.15 0.2 0.01"/>
+                    <box size="0.2 0.15 0.01"/>
                 </geometry>
             </visual>

File: bogobot_rviz/urdf/humanoid_main.urdf (robot description, URDF)
Before this commit: robot Bogobot_V1, 17 links, 16 joints
Links:
- added link link_left_foot; collision box size=0.2 0.15 0.01; visual box size=0.2 0.15 0.01
- added link link_right_foot; collision box size=0.2 0.15 0.01; visual box size=0.2 0.15 0.01
Joints:
- added joint q17: type revolute, parent link_right_ankle_motor, child link_right_foot, origin xyz=-0.02625 0.0 -0.01 rpy=0 0 0, axis 1 0 0, limit lower=-6.283185307179586 upper=6.283185307179586 effort=2.5 velocity=5.76
- added joint q18: type revolute, parent link_left_ankle_motor, child link_left_foot, origin xyz=0.02625 0.0 -0.01 rpy=0 0 0, axis 1 0 0, limit lower=-6.283185307179586 upper=6.283185307179586 effort=2.5 velocity=5.76

File: bogobot_rviz/urdf/humanoid_main.urdf.xacro (robot description, xacro)
@@ -19,4 +19,5 @@
     <xacro:link_knee name="link_right_knee" x = "0.0" y = "0.0" z = "-0.08" row = "0" pitch = "0" yaw = "0"/>
     <xacro:motor_big_double_join name="link_right_ankle_motor" x = "-0.02625" y = "0.0" z = "0.02" row = "0" pitch = "0" yaw = "0"/>
+    <xacro:foot name="link_right_foot" x = "0.025" y = "0.03" z = "0.0" row = "0" pitch = "0" yaw = "0"/>
     <!--pierna izquierda-->
     <xacro:hip_metal_link name="link_left_hip_metal" x = "0.0" y = "0.0" z = "-0.0175" row = "0" pitch = "0" yaw = "0"/>
@@ -25,4 +26,5 @@
     <xacro:link_knee name="link_left_knee" x = "0.0" y = "0.0" z = "-0.08" row = "0" pitch = "0" yaw = "0"/>
     <xacro:motor_big_double_join name="link_left_ankle_motor" x = "-0.02625" y = "0.0" z = "0.02" row = "0" pitch = "0" yaw = "0"/>
+    <xacro:foot name="link_left_foot" x = "-0.025" y = "-0.03" z = "0.0" row = "0" pitch = "0" yaw = "0"/>
     <!--JOINTS-->
     <!--hombro derecho-->
@@ -110,4 +112,11 @@
         <limit effort="2.5" lower="${-2*pi}" upper="${2*pi}" velocity="5.76"/>
     </joint>
+    <joint name="q17" type="revolute">
+        <origin rpy="0 0 0" xyz="-0.02625 0.0 -0.01" />
+        <parent link="link_right_ankle_motor" />
+        <child link="link_right_foot" />
+        <axis xyz="1 0 0" />
+        <limit effort="2.5" lower="${-2*pi}" upper="${2*pi}" velocity="5.76"/>
+    </joint>
     <!--pierna izquierda-->
     <joint name="q8" type="revolute">
@@ -146,3 +155,10 @@
         <limit effort="2.5" lower="${-2*pi}" upper="${2*pi}" velocity="5.76"/>
     </joint>
+    <joint name="q18" type="revolute">
+        <origin rpy="0 0 0" xyz="0.02625 0.0 -0.01" />
+        <parent link="link_left_ankle_motor" />
+        <child link="link_left_foot" />
+        <axis xyz="1 0 0" />
+        <limit effort="2.5" lower="${-2*pi}" upper="${2*pi}" velocity="5.76"/>
+    </joint>
 </robot>
